File: bridge_driver0_sch.kicad_sch (KiCad schematic)
At the start: 15 parts

Commit message: sdfgsdfs
Parts:
- JP?: value Jumper_3_Open -> SampleRate
- JP?: value Jumper_3_Open3 -> INB GND
Changed lines of the file:
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@@
   (symbol (lib_id "Jumper:Jumper_3_Open") (at 174.625 76.835 270)
     (in_bom yes) (on_board yes) (fields_autoplaced)
-    (property "Reference" "JP?" (id 0) (at 177.165 75.5649 90)
+    (property "Reference" "JP?" (id 0) (at 177.8 75.5649 90)
       (effects (font (size 1.27 1.27)) (justify left))
     )
-    (property "Value" "Jumper_3_Open" (id 1) (at 177.165 78.1049 90)
+    (property "Value" "SampleRate" (id 1) (at 177.8 78.1049 90)
       (effects (font (size 1.27 1.27)) (justify left))
     )
@@
   (symbol (lib_id "000_Connectors_Immo:Jumper_3_Open3") (at 164.465 102.235 180)
     (in_bom yes) (on_board yes) (fields_autoplaced)
-    (property "Reference" "JP?" (id 0) (at 169.545 101.0795 0)
+    (property "Reference" "JP?" (id 0) (at 168.91 101.0795 0)
       (effects (font (size 1.27 1.27)) (justify right))
     )
-    (property "Value" "Jumper_3_Open3" (id 1) (at 169.545 103.6195 0)
+    (property "Value" "INB GND" (id 1) (at 168.91 103.6195 0)
       (effects (font (size 1.27 1.27)) (justify right))
     )

Commit message: daily update
Parts:
- removed C? (x3): 100n, Capacitor_SMD:C_0805_2012Metric_Pad1.18x1.45mm_HandSolder, symbol 000_Capacitor_Film_Immo:cap_film_0805
- removed EC? (x2): 10u, Capacitor_SMD:CP_Elec_6.3x5.9, symbol 000_Capacitor_Electrolytic_Immo:22u
- removed J?: IN_B, Connector_PinHeader_1.27mm:PinHeader_1x02_P1.27mm_Vertical, symbol 000_Pin_Headers_Immo:Conn_01x02_Male
- removed JP?: Gain, Jumper:SolderJumper-2_P1.3mm_Open_RoundedPad1.0x1.5mm, symbol Jumper:Jumper_2_Open
- removed JP?: SampleRate, symbol Jumper:Jumper_3_Open
- removed JP?: INB GND, symbol 000_Connectors_Immo:Jumper_3_Open3
- removed Q?: BC807, Package_TO_SOT_SMD:SOT-23, symbol Transistor_BJT:BC807
- removed R? (x2): Resistor_0805, Resistor_SMD:R_0805_2012Metric_Pad1.20x1.40mm_HandSolder, symbol 000_Resistors_Immo:Resistor_0805
- removed R? (x2): 100r, Resistor_SMD:R_0805_2012Metric_Pad1.20x1.40mm_HandSolder, symbol 000_Resistors_Immo:Resistor_0805
- removed U?: HX711_24bit_ADC_Strain_Gauge_Driver, Package_SO:SOP-16_4.55x10.3mm_P1.27mm, symbol 000_Sensors_Immo:HX711_24bit_ADC_Strain_Gauge_Driver
- added C16, C17, C18: 100n, Capacitor_SMD:C_0805_2012Metric_Pad1.18x1.45mm_HandSolder, symbol 000_Capacitor_Film_Immo:cap_film_0805
- added EC11, EC12: 10u, Capacitor_SMD:CP_Elec_6.3x5.9, symbol 000_Capacitor_Electrolytic_Immo:22u
- added J10: IN_B, Connector_PinHeader_1.27mm:PinHeader_1x02_P1.27mm_Vertical, symbol 000_Pin_Headers_Immo:Conn_01x02_Male
- added JP17: Gain, Jumper:SolderJumper-2_P1.3mm_Bridged_RoundedPad1.0x1.5mm, symbol 000_Connectors_Immo:Jumper_2_Bridge_Small
- added JP18: INB GND, Jumper:SolderJumper-3_P1.3mm_Bridged12_RoundedPad1.0x1.5mm, symbol 000_Connectors_Immo:Jumper_3_BridgeSmall
- added JP19: Sample Rate, Jumper:SolderJumper-2_P1.3mm_Bridged_RoundedPad1.0x1.5mm, symbol 000_Connectors_Immo:Jumper_2_Bridge_Small
- added Q6: BC807, Package_TO_SOT_SMD:SOT-23, symbol Transistor_BJT:BC807
- added R27: 12k, Resistor_SMD:R_0805_2012Metric_Pad1.20x1.40mm_HandSolder, symbol 000_Resistors_Immo:Resistor_0805
- added R28: 33k, Resistor_SMD:R_0805_2012Metric_Pad1.20x1.40mm_HandSolder, symbol 000_Resistors_Immo:Resistor_0805
- added R29, R30: 100r, Resistor_SMD:R_0805_2012Metric_Pad1.20x1.40mm_HandSolder, symbol 000_Resistors_Immo:Resistor_0805
- added R31: 10k, Resistor_SMD:R_0805_2012Metric_Pad1.20x1.40mm_HandSolder, symbol 000_Resistors_Immo:Resistor_0805
- added U6: HX711_24bit_ADC_Strain_Gauge_Driver, Package_SO:SOP-16_4.55x10.3mm_P1.27mm, symbol 000_Sensors_Immo:HX711_24bit_ADC_Strain_Gauge_Driver
Connections:
- net 5V_DC: now also C18.1, EC12.1, Q6.2 (E), R31.1, U6.1 (Vdd), U6.16 (DVdd)
- net AGND: now also C16.2, C18.2, EC11.2, EC12.2, JP18.2 (C), JP19.1 (A), R28.1, U6.14 (XI), U6.5 (AGND)
- net CLK: now also U6.11 (PD_SCK)
- net D_OUT: now also U6.12 (Dout)
- net LC+: now also R30.2
- net LC-: now also R29.2
- net V_LC: now also EC11.1, JP17.2 (B), Q6.3 (C), R27.2
- new net: Q6.1 (B), U6.2 (Base)
- new net: C17.1, R29.1, U6.7 (INA-)
- new net: C17.2, R30.1, U6.8 (INA+)
- new net: J10.1 (Pin_1), JP18.1 (A), U6.9 (INB-)
- new net: J10.2 (Pin_2), JP18.3 (B), U6.10 (INB+)
- new net: JP19.2 (B), R31.2, U6.15 (Rate)
- new net: JP17.1 (A), U6.3 (AVdd)
- new net: R27.1, R28.2, U6.4 (VFB)
- new net: C16.1, U6.6 (VBG)
Other:
- note added: "Resistors: Vsup | R1 | R2 | 5v | 12k | 33k | 3.3v | 13k | 20k |"

Commit message: Daily Update
Parts:
- JP3: renamed from JP18; footprint Jumper:SolderJumper-3_P1.3mm_Bridged12_RoundedPad1.0x1.5mm -> Jumper:SolderJumper-3_P1.3mm_Bridged12_RoundedPad1.0x1.5mm_DoubleJoined_SMALL
- U1: renamed from U6; value HX711_24bit_ADC_Strain_Gauge_Driver -> HX711
- renumbered C16 to C1, C17 to C2, C18 to C3, EC11 to EC1, EC12 to EC2, J10 to J5, JP17 to JP2, JP19 to JP4, Q6 to Q1, R27 to R2, R28 to R3, R29 to R4, R30 to R5, R31 to R6
