File: micro_controller_sch.kicad_sch (KiCad schematic)
At the start: 0 parts

Commit message: daily update
Parts:
- added A1: Arduino_Nano_v3.x, Module:Arduino_Nano, symbol MCU_Module:Arduino_Nano_v3.x
- added C22, C23, C24, C25, C26, C27: 100n, Capacitor_SMD:C_0805_2012Metric_Pad1.18x1.45mm_HandSolder, symbol 000_Capacitor_Film_Immo:cap_film_0805
- added D1: LED, Diode_SMD:D_0805_2012Metric_Pad1.15x1.40mm_HandSolder, symbol 000_Diodes_Immo:LED_0805_smd
- added H1, H2, H3, H4: MountingHole_M3, MountingHole:MountingHole_3.2mm_M3_Pad_Via, symbol Mechanical:MountingHole_M3
- added J12: Serial IO, Connector_PinHeader_2.54mm:PinHeader_1x05_P2.54mm_Vertical, symbol 000_Pin_Headers_Immo:Conn_01x05_Male
- added J13: IO Header, Connector_PinHeader_2.54mm:PinHeader_1x08_P2.54mm_Vertical, symbol Connector:Conn_01x08_Male
- added J14: LV IO, Connector_PinHeader_2.54mm:PinHeader_1x05_P2.54mm_Vertical, symbol 000_Pin_Headers_Immo:Conn_01x05_Male
- added J15: HV IO, Connector_PinHeader_2.54mm:PinHeader_1x05_P2.54mm_Vertical, symbol 000_Pin_Headers_Immo:Conn_01x05_Male
- added JP26: V_USB, Jumper:SolderJumper-2_P1.3mm_Open_RoundedPad1.0x1.5mm, symbol 000_Connectors_Immo:Jumper_2_Open_small
- added JP27: 3v3, Jumper:SolderJumper-2_P1.3mm_Open_RoundedPad1.0x1.5mm, symbol 000_Connectors_Immo:Jumper_2_Open_small
- added JP28: 5v, Jumper:SolderJumper-2_P1.3mm_Open_RoundedPad1.0x1.5mm, symbol 000_Connectors_Immo:Jumper_2_Open_small
- added JP29: PWM, Jumper:SolderJumper-2_P1.3mm_Open_RoundedPad1.0x1.5mm, symbol 000_Connectors_Immo:Jumper_2_Open_small
- added JP30: DT1, Jumper:SolderJumper-2_P1.3mm_Open_RoundedPad1.0x1.5mm, symbol 000_Connectors_Immo:Jumper_2_Open_small
- added JP31: DT2, Jumper:SolderJumper-2_P1.3mm_Open_RoundedPad1.0x1.5mm, symbol 000_Connectors_Immo:Jumper_2_Open_small
- added JP32: DT3, Jumper:SolderJumper-2_P1.3mm_Open_RoundedPad1.0x1.5mm, symbol 000_Connectors_Immo:Jumper_2_Open_small
- added JP33: DT4, Jumper:SolderJumper-2_P1.3mm_Open_RoundedPad1.0x1.5mm, symbol 000_Connectors_Immo:Jumper_2_Open_small
- added JP34: DT5, Jumper:SolderJumper-2_P1.3mm_Open_RoundedPad1.0x1.5mm, symbol 000_Connectors_Immo:Jumper_2_Open_small
- added JP35: DT6, Jumper:SolderJumper-2_P1.3mm_Open_RoundedPad1.0x1.5mm, symbol 000_Connectors_Immo:Jumper_2_Open_small
- added JP36: DT7, Jumper:SolderJumper-2_P1.3mm_Open_RoundedPad1.0x1.5mm, symbol 000_Connectors_Immo:Jumper_2_Open_small
- added JP37: DT8, Jumper:SolderJumper-2_P1.3mm_Open_RoundedPad1.0x1.5mm, symbol 000_Connectors_Immo:Jumper_2_Open_small
- added JP38: LIM, Jumper:SolderJumper-2_P1.3mm_Open_RoundedPad1.0x1.5mm, symbol 000_Connectors_Immo:Jumper_2_Open_small
- added JP39: SCK, Jumper:SolderJumper-2_P1.3mm_Open_RoundedPad1.0x1.5mm, symbol 000_Connectors_Immo:Jumper_2_Open_small
- added R37: 1k, Resistor_SMD:R_0805_2012Metric_Pad1.20x1.40mm_HandSolder, symbol 000_Resistors_Immo:Resistor_0805
- added U8, U9: TXS0108EPW, Package_SO:TSSOP-20_4.4x6.5mm_P0.65mm, symbol Logic_LevelTranslator:TXS0108EPW
Connections:
- new net: J15.1 (Pin_1), U8.12 (B8)
- new net: J15.2 (Pin_2), U8.13 (B7)
- new net: J15.3 (Pin_3), U8.14 (B6)
- new net: J15.4 (Pin_4), U8.15 (B5)
- new net: J15.5 (Pin_5), U8.16 (B4)
- new net: J14.1 (Pin_1), U8.5 (A4)
- new net: J14.2 (Pin_2), U8.6 (A5)
- new net: J14.3 (Pin_3), U8.7 (A6)
- new net: J14.4 (Pin_4), U8.8 (A7)
- new net: J14.5 (Pin_5), U8.9 (A8)
- new net: D1.1 (K), R37.2
- new net: A1.17 (3V3), JP27.1 (A)
- new net: A1.30 (VIN), JP26.1 (A)
- new net: A1.1 (D1/TX), J12.5 (Pin_5)
- new net: A1.19 (A0), J13.1 (Pin_1)
- new net: A1.2 (D0/RX), J12.4 (Pin_4)
- new net: A1.21 (A2), J13.2 (Pin_2)
- new net: A1.22 (A3), J13.3 (Pin_3)
- new net: A1.23 (A4), J13.4 (Pin_4)
- new net: A1.24 (A5), J13.5 (Pin_5)
- new net: A1.25 (A6), J13.6 (Pin_6)
- new net: A1.26 (A7), J13.7 (Pin_7)
- new net: A1.27 (+5V), JP28.1 (A)
- new net 3V3_VDC: C22.1, C24.1, C25.1, JP27.2 (B), U8.2 (VCCA), U9.2 (VCCA)
- new net 5__VDC: C23.1, C26.1, C27.1, JP28.2 (B), U8.19 (VCCB), U9.19 (VCCB)
- new net DGND: A1.29 (GND), A1.4 (GND), C22.2, C23.2, C24.2, C25.2, C26.2, C27.2, J12.1 (Pin_1), R37.1, U8.11 (GND), U9.11 (GND)
- new net DT1: A1.6 (D3), JP30.1 (A), JP30.2 (B), U9.1 (A1), U9.20 (B1)
- new net DT2: A1.7 (D4), JP31.1 (A), JP31.2 (B), U9.18 (B2), U9.3 (A2)
- new net DT3: A1.8 (D5), JP32.1 (A), JP32.2 (B), U9.17 (B3), U9.4 (A3)
- new net DT4: A1.9 (D6), JP33.1 (A), JP33.2 (B), U9.16 (B4), U9.5 (A4)
- new net DT5: A1.10 (D7), JP34.1 (A), JP34.2 (B), U9.15 (B5), U9.6 (A5)
- new net DT6: A1.11 (D8), JP35.1 (A), JP35.2 (B), U9.14 (B6), U9.7 (A6)
- new net DT7: A1.12 (D9), JP36.1 (A), JP36.2 (B), U9.13 (B7), U9.8 (A7)
- new net DT8: A1.13 (D10), JP37.1 (A), JP37.2 (B), U9.12 (B8), U9.9 (A8)
- new net LIMIT_SWITCH: A1.14 (D11), JP38.1 (A), JP38.2 (B), U8.17 (B3), U8.4 (A3)
- new net OUTPUT_ENABLE: A1.20 (A1), U8.10 (OE), U9.10 (OE)
- new net RST: A1.28 (~{RESET}), A1.3 (~{RESET}), J12.3 (Pin_3)
- new net SCK: A1.5 (D2), JP39.1 (A), JP39.2 (B), U8.18 (B2), U8.3 (A2)
- new net SERVO_PWM_OUTPUT: JP29.1 (A), U8.20 (B1)
- new net SERVO_PWM_PIN: A1.15 (D12), JP29.2 (B), U8.1 (A1)
- new net SPARE_0: A1.16 (D13), D1.2 (A), J13.8 (Pin_8)
- new net V_USB: J12.2 (Pin_2), JP26.2 (B)
- no-connect marks 0 -> 1
Other:
- note added: "Logic Level Shifter only required for use with 3v3 MCU"

Commit message: Daily Update
Parts:
- added D10, D11, D9: LED, Diode_SMD:D_0805_2012Metric_Pad1.15x1.40mm_HandSolder, symbol 000_Diodes_Immo:LED_0805_smd
- added R44, R45, R46: 1k, Resistor_SMD:R_0805_2012Metric_Pad1.20x1.40mm_HandSolder, symbol 000_Resistors_Immo:Resistor_0805
- JP30: value DT1 -> DT0
- JP31: value DT2 -> DT1
- JP32: value DT3 -> DT2
- JP33: value DT4 -> DT3
- JP34: value DT5 -> DT4
- JP35: value DT6 -> DT5
- JP36: value DT7 -> DT6
- JP37: value DT8 -> DT7
Connections:
- net DGND: now also R44.1, R45.1, R46.1
- net DT1: now also A1.7 (D4), JP31.2 (B), U9.3 (A2); no longer A1.6 (D3), JP30.1 (A), JP30.2 (B), U9.1 (A1), U9.20 (B1)
- net DT2: now also A1.8 (D5), JP32.2 (B), U9.4 (A3); no longer A1.7 (D4), JP31.1 (A), JP31.2 (B), U9.18 (B2), U9.3 (A2)
- net DT3: now also A1.9 (D6), JP33.2 (B), U9.5 (A4); no longer A1.8 (D5), JP32.1 (A), JP32.2 (B), U9.17 (B3), U9.4 (A3)
- net DT4: now also A1.10 (D7), JP34.2 (B), U9.6 (A5); no longer A1.9 (D6), JP33.1 (A), JP33.2 (B), U9.16 (B4), U9.5 (A4)
- net DT5: now also A1.11 (D8), JP35.2 (B), U9.7 (A6); no longer A1.10 (D7), JP34.1 (A), JP34.2 (B), U9.15 (B5), U9.6 (A5)
- net DT6: now also A1.12 (D9), JP36.2 (B), U9.8 (A7); no longer A1.11 (D8), JP35.1 (A), JP35.2 (B), U9.14 (B6), U9.7 (A6)
- net DT7: now also A1.13 (D10), JP37.2 (B), U9.9 (A8); no longer A1.12 (D9), JP36.1 (A), JP36.2 (B), U9.13 (B7), U9.8 (A7)
- net LIMIT_SWITCH: no longer JP38.1 (A), U8.17 (B3)
- net SCK: no longer JP39.1 (A), U8.18 (B2)
- net at A1.24 (A5), J13.5 (Pin_5): now also D9.2 (A)
- net at A1.25 (A6), J13.6 (Pin_6): now also D10.2 (A)
- net at A1.26 (A7), J13.7 (Pin_7): now also D11.2 (A)
- removed net DT8: A1.13 (D10), JP37.1 (A), JP37.2 (B), U9.12 (B8), U9.9 (A8)
- net SERVO_PWM_OUTPUT renamed SERVO_PWM_OUT
- new net: D11.1 (K), R46.2
- new net: D10.1 (K), R45.2
- new net: D9.1 (K), R44.2
- new net DATA_0: JP30.1 (A), U9.20 (B1)
- new net DATA_1: JP31.1 (A), U9.18 (B2)
- new net DATA_2: JP32.1 (A), U9.17 (B3)
- new net DATA_3: JP33.1 (A), U9.16 (B4)
- new net DATA_4: JP34.1 (A), U9.15 (B5)
- new net DATA_5: JP35.1 (A), U9.14 (B6)
- new net DATA_6: JP36.1 (A), U9.13 (B7)
- new net DATA_7: JP37.1 (A), U9.12 (B8)
- new net DT0: A1.6 (D3), JP30.2 (B), U9.1 (A1)
- new net LIMIT_SWITCH_IN: JP38.1 (A), U8.17 (B3)
- new net SCK_OUT: JP39.1 (A), U8.18 (B2)
Other:
- moved on the sheet: J13
