File: load_cell.kicad_sch (KiCad schematic)
At the start: 0 parts

Commit message: sdfgsdfs
Parts:
- added C? (x3): 100n, Capacitor_SMD:C_0805_2012Metric_Pad1.18x1.45mm_HandSolder, symbol 000_Capacitor_Film_Immo:cap_film_0805
- added EC? (x2): 10u, Capacitor_SMD:CP_Elec_6.3x5.9, symbol 000_Capacitor_Electrolytic_Immo:22u
- added J?: IN_B, Connector_PinHeader_1.27mm:PinHeader_1x02_P1.27mm_Vertical, symbol 000_Pin_Headers_Immo:Conn_01x02_Male
- added JP?: LC Vsup, symbol 000_Connectors_Immo:Jumper_3_Open3small
- added JP?: Gain, Jumper:SolderJumper-2_P1.3mm_Open_RoundedPad1.0x1.5mm, symbol 000_Connectors_Immo:Jumper_2_Open_small
- added JP?: SampleRate, Jumper:SolderJumper-2_P1.3mm_Open_RoundedPad1.0x1.5mm, symbol 000_Connectors_Immo:Jumper_2_Open_small
- added JP?: INB GND, symbol 000_Connectors_Immo:Jumper_3_Open3small
- added JP?: Base, Jumper:SolderJumper-2_P1.3mm_Open_RoundedPad1.0x1.5mm, symbol 000_Connectors_Immo:Jumper_2_Open_small
- added JP?: VFB, Jumper:SolderJumper-2_P1.3mm_Open_RoundedPad1.0x1.5mm, symbol 000_Connectors_Immo:Jumper_2_Open_small
- added Q?: BC807, Package_TO_SOT_SMD:SOT-23, symbol Transistor_BJT:BC807
- added R? (x2): 100r, Resistor_SMD:R_0805_2012Metric_Pad1.20x1.40mm_HandSolder, symbol 000_Resistors_Immo:Resistor_0805
- added R?: 12k, Resistor_SMD:R_0805_2012Metric_Pad1.20x1.40mm_HandSolder, symbol 000_Resistors_Immo:Resistor_0805
- added R?: 10k, Resistor_SMD:R_0805_2012Metric_Pad1.20x1.40mm_HandSolder, symbol 000_Resistors_Immo:Resistor_0805
- added R?: 33k, Resistor_SMD:R_0805_2012Metric_Pad1.20x1.40mm_HandSolder, symbol 000_Resistors_Immo:Resistor_0805
- added U?: HX711_24bit_ADC_Strain_Gauge_Driver, Package_SO:SOP-16_4.55x10.3mm_P1.27mm, symbol 000_Sensors_Immo:HX711_24bit_ADC_Strain_Gauge_Driver
Connections:
- new net: JP?.2 (B), Q?.1 (B)
- new net: EC?.1, JP?.1 (A), JP?.2 (B), Q?.3 (C), R?.2
- new net: J?.2 (Pin_2), JP?.3 (B), U?.10 (INB+)
- new net: JP?.2 (B), R?.2, U?.15 (Rate)
- new net: JP?.1 (A), U?.2 (Base)
- new net: JP?.1 (A), U?.3 (AVdd)
- new net: JP?.1 (A), R?.1, R?.2, U?.4 (VFB)
- new net: C?.1, U?.6 (VBG)
- new net: C?.1, R?.1, U?.7 (INA-)
- new net: C?.2, R?.1, U?.8 (INA+)
- new net: J?.1 (Pin_1), JP?.1 (A), U?.9 (INB-)
- new net 10V_DC: JP?.3 (B)
- new net 5V_DC: C?.1, EC?.1, Q?.2 (E), R?.1, U?.1 (Vdd), U?.16 (DVdd)
- new net AGND: C?.2, C?.2, EC?.2, EC?.2, JP?.1 (A), JP?.2 (B), JP?.2 (C), R?.1, U?.14 (XI), U?.5 (AGND)
- new net CLK: U?.11 (PD_SCK)
- new net D_OUT: U?.12 (Dout)
- new net LC+: R?.2
- new net LC-: R?.2
- new net V_LC: JP?.2 (C)
- no-connect marks 0 -> 1
Other:
- note added: "CH A Jumper | Gain | Input Range -----|----|------ Open | 128 | +-20mA Short | 64 | +-40mA CH B Gain 32"
- note added: "If using EXTERNAL excitation Voltage: Base - OPEN VFB - SHORTED - GND Resistors - Omit VBG Cap - Omit"
- note added: "Jumper | Sample Rate -----|------- Vcc | 80Hz GND | 10Hz"
- note added: "Resistors: Vsup | R1 | R2 | 5v | 12k | 33k | 3.3v | 13k | 20k |"

Commit message: daily update
Parts:
- removed JP?: Gain, Jumper:SolderJumper-2_P1.3mm_Open_RoundedPad1.0x1.5mm, symbol 000_Connectors_Immo:Jumper_2_Open_small
- removed JP?: INB GND, symbol 000_Connectors_Immo:Jumper_3_Open3small
- removed JP?: Base, Jumper:SolderJumper-2_P1.3mm_Open_RoundedPad1.0x1.5mm, symbol 000_Connectors_Immo:Jumper_2_Open_small
- added JP21: Gain, Jumper:SolderJumper-2_P1.3mm_Bridged_RoundedPad1.0x1.5mm, symbol 000_Connectors_Immo:Jumper_2_Bridge_Small
- added JP23: Base, Jumper:SolderJumper-2_P1.3mm_Bridged_RoundedPad1.0x1.5mm, symbol 000_Connectors_Immo:Jumper_2_Bridge_Small
- added JP24: INB GND, Jumper:SolderJumper-3_P1.3mm_Bridged12_RoundedPad1.0x1.5mm, symbol 000_Connectors_Immo:Jumper_3_BridgeSmall
- JP20: renamed from JP?; footprint (none) -> Jumper:SolderJumper-3_P1.3mm_Open_RoundedPad1.0x1.5mm_NumberLabels
- gave numbers to parts that had none: 15
Connections:
- net AGND: now also JP24.2 (C)
- net at Q7.1 (B): now also JP23.2 (B)
- net at EC13.1, JP20.1 (A), Q7.3 (C)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: now also JP21.2 (B)
- net at J11.2 (Pin_2), U7.10 (INB+): now also JP24.3 (B)
- net at U7.2 (Base): now also JP23.1 (A)
- net at U7.3 (AVdd): now also JP21.1 (A)
- net at J11.1 (Pin_1), U7.9 (INB-): now also JP24.1 (A)

Commit message: Daily Update
Parts:
- JP24: footprint Jumper:SolderJumper-3_P1.3mm_Bridged12_RoundedPad1.0x1.5mm -> Jumper:SolderJumper-3_P1.3mm_Bridged12_RoundedPad1.0x1.5mm_DoubleJoined_SMALL
- U7: value HX711_24bit_ADC_Strain_Gauge_Driver -> HX711
Changed lines of the file:
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@@
     (in_bom yes) (on_board yes)
     (property "Reference" "U7" (id 0) (at 147.955 62.23 0))
-    (property "Value" "HX711_24bit_ADC_Strain_Gauge_Driver" (id 1) (at 147.955 64.77 0))
+    (property "Value" "HX711" (id 1) (at 147.955 64.77 0))
     (property "Footprint" "Package_SO:SOP-16_4.55x10.3mm_P1.27mm" (id 2) (at 134.62 115.57 0)
       (effects (font (size 1.27 1.27) italic) (justify left) hide)
@@
       (effects (font (size 1.27 1.27)) (justify left))
     )
-    (property "Footprint" "Jumper:SolderJumper-3_P1.3mm_Bridged12_RoundedPad1.0x1.5mm" (id 2) (at 163.195 102.235 0)
-      (effects (font (size 1.27 1.27)) hide)
-    )
+    (property "Footprint" "Jumper:SolderJumper-3_P1.3mm_Bridged12_RoundedPad1.0x1.5mm_DoubleJoined_SMALL" (id 2) (at 163.195 102.235 0)
+      (effects (font (size 1.27 1.27)) hide)
+    )

Commit message: Added lots of files
Parts:
- JP25: footprint Jumper:SolderJumper-2_P1.3mm_Open_RoundedPad1.0x1.5mm -> Jumper:SolderJumper-2_P1.3mm_Bridged_RoundedPad1.0x1.5mm; symbol 000_Connectors_Immo:Jumper_2_Open_small -> 000_Connectors_Immo:Jumper_2_Bridge_Small
Changed lines of the file:
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@@
     (pin "2")
   )
-  (symbol (lib_id "000_Connectors_Immo:Jumper_2_Open_small") (at 173.99 80.645 90) (unit 1)
+  (symbol (lib_id "000_Connectors_Immo:Jumper_2_Bridge_Small") (at 173.99 80.645 90) (unit 1)
     (in_bom yes) (on_board yes) (fields_autoplaced)
     (property "Reference" "JP25" (id 0) (at 176.53 79.6903 90)
@@
       (effects (font (size 1.27 1.27)) (justify right))
     )
-    (property "Footprint" "Jumper:SolderJumper-2_P1.3mm_Open_RoundedPad1.0x1.5mm" (id 2) (at 179.705 80.01 0)
+    (property "Footprint" "Jumper:SolderJumper-2_P1.3mm_Bridged_RoundedPad1.0x1.5mm" (id 2) (at 179.705 80.01 0)
       (effects (font (size 1.27 1.27)) hide)
     )
