File: truss_PCB.kicad_pcb (KiCad board)
At the start: 2 copper layers, 99.1 x 99.1 mm, 190 parts, among them IC1 BAJ0BC0FP-E2, J1 XT60_60A_male, J10 IN_B, J11 IN_B, J12 Serial IO, J13 IO Header, J14 LV IO, J15 HV IO, J2 LimitSwitch, J3 Servo, J4 Truss Connection, J5 IN_B, J6 IN_B, J7 IN_B, J8 IN_B, J9 IN_B, Q1 BC807, Q2 BC807, Q3 BC807, Q4 BC807, Q5 BC807, Q6 BC807, Q7 BC807, Q8 IRF5305_PBF, U1 HX711_24bit_ADC_Strain_Gauge_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, U10 R-78E5.0-1.0, U11 LM2596S-ADJ, U12 AMS1117-5.0, U13 AMS1117-3.3, U2 HX711_24bit_ADC_Strain_Gauge_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, U3 HX711_24bit_ADC_Strain_Gauge_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, U4 HX711_24bit_ADC_Strain_Gauge_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, U5 HX711_24bit_ADC_Strain_Gauge_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, U6 HX711_24bit_ADC_Strain_Gauge_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, U7 HX711_24bit_ADC_Strain_Gauge_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, U8 TXS0108EPW, U9 TXS0108EPW

Commit message: Daily Update
Parts:
- removed C29: 220u, Capacitor_SMD:CP_Elec_6.3x7.7
- removed EC16: 10u, Capacitor_SMD:CP_Elec_6.3x5.9
- removed N1: pwr_tie, NetTie:NetTie-8-15A_1oz_2oz
- removed U10: R-78E5.0-1.0, Converter_DCDC:Converter_DCDC_RECOM_R-78E-0.5_THT
- added D10: LED, Diode_SMD:D_0805_2012Metric_Pad1.15x1.40mm_HandSolder, F.Cu at (124.5, 132.7)
- added D11: LED, Diode_SMD:D_0805_2012Metric_Pad1.15x1.40mm_HandSolder, F.Cu at (127.6, 132.7)
- added D9: LED, Diode_SMD:D_0805_2012Metric_Pad1.15x1.40mm_HandSolder, F.Cu at (121.3, 132.7)
- added N3: pwr_tie, NetTie:NetTie-8-15A_1oz_2oz, F.Cu at (104.8, 109.4)
- added R44: 1k, Resistor_SMD:R_0805_2012Metric_Pad1.20x1.40mm_HandSolder, F.Cu at (121.3, 123.5)
- added R45: 1k, Resistor_SMD:R_0805_2012Metric_Pad1.20x1.40mm_HandSolder, F.Cu at (124.5, 123.5)
- added R46: 1k, Resistor_SMD:R_0805_2012Metric_Pad1.20x1.40mm_HandSolder, F.Cu at (127.6, 123.5)
- C28: footprint Capacitor_THT:C_Radial_D12.5mm_H20.0mm_P5.00mm -> Capacitor_SMD:CP_Elec_10x10
- D6: value 12V Power -> 10V Power
- EC15: value 22u -> 100u; footprint Capacitor_SMD:CP_Elec_6.3x5.9 -> Capacitor_SMD:CP_Elec_10x10
- JP10, JP11, JP13, JP14, JP16, JP17, JP19, JP2, JP20, JP21, JP22, JP23, JP25, JP4, JP5, JP7, JP8: moved to B.Cu
- JP12, JP15, JP18, JP24, JP3, JP6, JP9: footprint Jumper:SolderJumper-3_P1.3mm_Bridged12_RoundedPad1.0x1.5mm -> Jumper:SolderJumper-3_P1.3mm_Bridged12_RoundedPad1.0x1.5mm_DoubleJoined_SMALL; moved to B.Cu
- JP30: value DT1 -> DT0
- JP31: value DT2 -> DT1
- JP32: value DT3 -> DT2
- JP33: value DT4 -> DT3
- JP34: value DT5 -> DT4
- JP35: value DT6 -> DT5
- JP36: value DT7 -> DT6
- JP37: value DT8 -> DT7
- U1, U2, U3, U4, U5, U6, U7: value HX711_24bit_ADC_Strain_Gauge_Driver -> HX711
- moved C21 361.6 mm to (179.7, 137.8), turned to 180 degrees
- moved R36 357.9 mm to (181.6, 134.3), turned to -90 degrees
- moved JP21 356.2 mm to (188.0, 135.2), turned to 90 degrees
- moved JP23 354.6 mm to (191.1, 136.5)
- moved EC14 351.6 mm to (175.3, 132.7), turned to 90 degrees
- moved JP22 350.6 mm to (187.3, 132.1), turned to 180 degrees
- moved JP25 347.9 mm to (186.7, 138.4), turned to 180 degrees
- moved J11 344.3 mm to (181.0, 128.9)
- moved Q7 343.0 mm to (194.3, 138.4)
- moved R32 340.1 mm to (194.3, 135.3)
- moved R35 336.0 mm to (197.2, 127.6)
- moved JP24 335.7 mm to (186.7, 129.3), turned to -90 degrees
- moved C20 334.5 mm to (193.0, 128.7), turned to 90 degrees
- moved C19 334.3 mm to (186.5, 127.6), turned to 180 degrees
- moved C15 332.9 mm to (175.5, 111.1), turned to 180 degrees
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Connections:
- A1 pad 10: /MCU/DT5 -> /MCU/DT4
- A1 pad 11: /MCU/DT6 -> /MCU/DT5
- A1 pad 12: /MCU/DT7 -> /MCU/DT6
- A1 pad 13: /MCU/DT8 -> /MCU/DT7
- A1 pad 14: /LIMIT_SWITCH -> /MCU/LIMIT_SWITCH
- A1 pad 29: GNDD -> GNDA
- A1 pad 4: GNDD -> GNDA
- A1 pad 5: SCK -> /MCU/SCK
- A1 pad 6: /MCU/DT1 -> /MCU/DT0
- A1 pad 7: /MCU/DT2 -> /MCU/DT1
- A1 pad 8: /MCU/DT3 -> /MCU/DT2
- A1 pad 9: /MCU/DT4 -> /MCU/DT3
- C22 pad 2: GNDD -> GNDA
- C23 pad 2: GNDD -> GNDA
- C24 pad 2: GNDD -> GNDA
- C25 pad 2: GNDD -> GNDA
- C26 pad 2: GNDD -> GNDA
- C27 pad 2: GNDD -> GNDA
- EC15 pad 1: /Power Distribution/12V_BUS -> /SERVO_POWER
- J12 pad 1: GNDD -> GNDA
- J2 pad 1: GNDD -> GNDA
- J3 pad 3: GNDPWR -> /SERVO_GND
- J4 pad 0: GNDD -> GNDA
- J4 pad 19: GNDPWR -> /SERVO_GND
- J4 pad 36: GNDD -> GNDA
- JP30 pad 1: /MCU/DT1 -> /BridgeDriver0/D_OUT
- JP30 pad 2: /MCU/DT1 -> /MCU/DT0
- JP31 pad 1: /MCU/DT2 -> /BridgeDriver1/D_OUT
- JP31 pad 2: /MCU/DT2 -> /MCU/DT1
- JP32 pad 1: /MCU/DT3 -> /BridgeDriver2/D_OUT
- JP32 pad 2: /MCU/DT3 -> /MCU/DT2
- JP33 pad 1: /MCU/DT4 -> /BridgeDriver3/D_OUT
- JP33 pad 2: /MCU/DT4 -> /MCU/DT3
- JP34 pad 1: /MCU/DT5 -> /BridgeDriver4/D_OUT
- JP34 pad 2: /MCU/DT5 -> /MCU/DT4
- JP35 pad 1: /MCU/DT6 -> /BridgeDriver5/D_OUT
- JP35 pad 2: /MCU/DT6 -> /MCU/DT5
- JP36 pad 1: /MCU/DT7 -> /LoadCell/D_OUT
- JP36 pad 2: /MCU/DT7 -> /MCU/DT6
- JP37 pad 1: /MCU/DT8 -> /MCU/DATA_7
- JP37 pad 2: /MCU/DT8 -> /MCU/DT7
- JP38 pad 2: /LIMIT_SWITCH -> /MCU/LIMIT_SWITCH
- JP39 pad 2: SCK -> /MCU/SCK
- N2 pad 1: GNDD -> GNDA
- N2 pad 2: GNDA -> GNDPWR
- R37 pad 1: GNDD -> GNDA
- U1 pad 12: /MCU/DT1 -> /BridgeDriver0/D_OUT
- U2 pad 12: /MCU/DT2 -> /BridgeDriver1/D_OUT
- U3 pad 12: /MCU/DT3 -> /BridgeDriver2/D_OUT
- U4 pad 12: /MCU/DT4 -> /BridgeDriver3/D_OUT
- U5 pad 12: /MCU/DT5 -> /BridgeDriver4/D_OUT
- U6 pad 12: /MCU/DT6 -> /BridgeDriver5/D_OUT
- U7 pad 12: /MCU/DT7 -> /LoadCell/D_OUT
- U8 pad 11: GNDD -> GNDA
- U8 pad 3: SCK -> /MCU/SCK
- U8 pad 4: /LIMIT_SWITCH -> /MCU/LIMIT_SWITCH
- U9 pad 1: /MCU/DT1 -> /MCU/DT0
- U9 pad 11: GNDD -> GNDA
- U9 pad 12: /MCU/DT8 -> /MCU/DATA_7
- U9 pad 13: /MCU/DT7 -> /LoadCell/D_OUT
- U9 pad 14: /MCU/DT6 -> /BridgeDriver5/D_OUT
- U9 pad 15: /MCU/DT5 -> /BridgeDriver4/D_OUT
- U9 pad 16: /MCU/DT4 -> /BridgeDriver3/D_OUT
- U9 pad 17: /MCU/DT3 -> /BridgeDriver2/D_OUT
- U9 pad 18: /MCU/DT2 -> /BridgeDriver1/D_OUT
- U9 pad 20: /MCU/DT1 -> /BridgeDriver0/D_OUT
- U9 pad 3: /MCU/DT2 -> /MCU/DT1
- U9 pad 4: /MCU/DT3 -> /MCU/DT2
- U9 pad 5: /MCU/DT4 -> /MCU/DT3
- U9 pad 6: /MCU/DT5 -> /MCU/DT4
- U9 pad 7: /MCU/DT6 -> /MCU/DT5
- U9 pad 8: /MCU/DT7 -> /MCU/DT6
- U9 pad 9: /MCU/DT8 -> /MCU/DT7
Routing:
- net 5VDC: track 0.00 -> 470.2 mm, vias 0 -> 21
- net /SERVO_POWER: track 0.00 -> 257.7 mm, vias 0 -> 3
- net GNDA: track 0.00 -> 211.0 mm, vias 0 -> 60
- net /10V_DC: track 0.00 -> 205.5 mm, vias 0 -> 3
- net 3V3DC: track 0.00 -> 193.1 mm, vias 0 -> 4
- net SCK: track 0.00 -> 177.8 mm, vias 0 -> 2
- net /SERVO_GND: track 0.00 -> 176.2 mm
- net GNDPWR: track 0.00 -> 162.7 mm, vias 0 -> 41
- net /Power Distribution/12V_BUS: track 0.00 -> 140.0 mm
- net /MCU/OUTPUT_ENABLE: track 0.00 -> 123.3 mm, vias 0 -> 2
- net /LIMIT_SWITCH: track 0.00 -> 99.2 mm
- net /BridgeDriver0/D_OUT: track 0.00 -> 82.6 mm, vias 0 -> 2
- net /MCU/SERVO_PWM_PIN: track 0.00 -> 71.5 mm, vias 0 -> 2
- net /BridgeDriver1/D_OUT: track 0.00 -> 70.1 mm, vias 0 -> 4
- net /MCU/LIMIT_SWITCH: track 0.00 -> 68.0 mm, vias 0 -> 4
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- added copper zone on B.Cu, net GNDA
- added copper zone on B.Cu, net GNDPWR
Other:
- board size 99.1 x 99.1 mm -> 114.3 x 102.9 mm
- board text added: "10v PSU"
- board text added: "3v3 MCU PSU"
- board text added: "5v MCU PSU"
- board text added: "6v Servo PSU"
- board text added: "CH0"
- board text added: "CH1"
- board text added: "CH2"
- board text added: "CH3"
- board text added: "CH4"
- board text added: "CH5"
- board text added: "LC6"

Commit message: Added lots of files
Parts:
- added G***: LOGO, 000_Graphics_Immo:practactable.io_text_20x8, F.Cu at (144.3, 93.2)
- added G***: LOGO, 000_Graphics_Immo:practactable.io_text_80x30, B.Cu at (159.4, 94.0)
- JP25: footprint Jumper:SolderJumper-2_P1.3mm_Open_RoundedPad1.0x1.5mm -> Jumper:SolderJumper-2_P1.3mm_Bridged_RoundedPad1.0x1.5mm
- moved N2 0.35 mm to (157.1, 65.3)
- moved C23 0.23 mm to (131.4, 132.7)
Routing:
- net GNDA: track 211.0 -> 212.2 mm
- net /LoadCell/LC+: track 38.5 -> 39.0 mm
Other:
- board text added: "CH6"
- board text added: "Ex+"
- board text added: "GND"
- board text added: "LC+"
- board text added: "LC-"
- board text added: "LIM"
- board text added: "PWM"
- board text added: "Power"
- board text added: "RemoteLabs MiniTruss V1.0"
- board text added: "SERVO"
- board text added: "github.com/ImogenWren"
- board text added: "github.com/practable/minitruss"
