File: truss_PCB.kicad_sch (KiCad schematic)
At the start: 0 parts

Commit message: sdfgsdfs
Other:
- sheet LoadCell ports: added 10V_DC, 5V_DC, AGND, CLK, D_OUT, GND_LC, LC+, LC-, V_LC; removed none

Commit message: daily update
Parts:
- added J1: XT60_60A_male, Connector_AMASS:AMASS_XT60PW-M, symbol 000_Connectors_Immo:XT60_60A_male
- added J2: LimitSwitch, Connector_Molex:Molex_KK-254_AE-6410-02A_1x02_P2.54mm_Vertical, symbol 000_Connectors_Immo:2pin_molex_2.54mm_male
- added J3: Servo, Connector_PinHeader_2.54mm:PinHeader_1x03_P2.54mm_Vertical, symbol Connector:Conn_01x03_Male
- added J4: Truss Connection, Connector_Dsub:DSUB-37_Female_Vertical_P2.77x2.84mm_MountingHoles, symbol Connector:DB37_Female_MountingHoles
- added JP1: PWM_CONN, Jumper:SolderJumper-2_P1.3mm_Open_RoundedPad1.0x1.5mm, symbol 000_Connectors_Immo:Jumper_2_Open_small
- added N1, N2: pwr_tie, NetTie:NetTie-8-15A_1oz_2oz, symbol 000_Utility_Immo:pwr_tie
- added R1: 10k, Resistor_SMD:R_0805_2012Metric_Pad1.20x1.40mm_HandSolder, symbol 000_Resistors_Immo:Resistor_0805
Connections:
- net BridgeDriver0/GND_LC: now also J4.20
- net BridgeDriver0/LC+: now also J4.21
- net BridgeDriver0/LC-: now also J4.2
- net BridgeDriver0/V_LC: now also J4.1
- net BridgeDriver1/GND_LC: now also J4.22
- net BridgeDriver1/LC+: now also J4.23
- net BridgeDriver1/LC-: now also J4.4
- net BridgeDriver1/V_LC: now also J4.3
- net BridgeDriver2/GND_LC: now also J4.24
- net BridgeDriver2/LC+: now also J4.25
- net BridgeDriver2/LC-: now also J4.6
- net BridgeDriver2/V_LC: now also J4.5
- net BridgeDriver3/GND_LC: now also J4.26
- net BridgeDriver3/LC+: now also J4.27
- net BridgeDriver3/LC-: now also J4.8
- net BridgeDriver3/V_LC: now also J4.7
- net BridgeDriver4/GND_LC: now also J4.28
- net BridgeDriver4/LC+: now also J4.29
- net BridgeDriver4/LC-: now also J4.10
- net BridgeDriver4/V_LC: now also J4.9
- net BridgeDriver5/GND_LC: now also J4.30
- net BridgeDriver5/LC+: now also J4.31
- net BridgeDriver5/LC-: now also J4.12
- net BridgeDriver5/V_LC: now also J4.11
- net LoadCell/GND_LC: now also J4.32
- net LoadCell/LC+: now also J4.33
- net LoadCell/LC-: now also J4.14
- net LoadCell/V_LC: now also J4.13
- new net 5VDC: R1.2
- new net GNDA: N2.2 (C)
- new net GNDD: J2.1 (Pin_1), J4.0 (PAD), J4.36, N1.2 (C), N2.1 (A)
- new net GNDPWR: J1.1 (V-), J3.3 (Pin_3), J4.19, N1.1 (A)
- new net LIMIT_SWITCH: J2.2 (Pin_2), J4.17, R1.1
- new net PWM: J4.18, JP1.1 (A)
- new net Power Distribution/12V_IN: J1.2 (V+)
- new net SERVO_POWER: J3.2 (Pin_2), J4.37
- new net SERVO_PWM: J3.1 (Pin_1), JP1.2 (B)
- no-connect marks 0 -> 6
Other:
- removed sheet Actuator
- removed sheet BridgeDriver6
- sheet MCU ports: added 3V3_VDC, 5__VDC, DGND, DT1, DT2, DT3, DT4, DT5, DT6, DT7, DT8, LIMIT_SWITCH, SCK, SERVO_PWM_OUTPUT, V_USB; removed none
- sheet Power Distribution ports: added 10V_LC, 12V_IN, 3V3_MCU, 5V_MCU, 6V_SERVO, P_GND; removed none
- note added: "IN an ideal world, all signals go through big header However, provision in case PWM noise affects sensor readings to remove PWM from nearby analog signal lines"

Commit message: Daily Update
Parts:
- removed N1: pwr_tie, NetTie:NetTie-8-15A_1oz_2oz, symbol 000_Utility_Immo:pwr_tie
- added N3: pwr_tie, NetTie:NetTie-8-15A_1oz_2oz, symbol 000_Utility_Immo:pwr_tie
Connections:
- net GNDD is gone; now on net GNDA: J2.1 (Pin_1), J4.0 (PAD), J4.36, N2.1 (A)
- net GNDA: no longer N2.2 (C)
- net GNDPWR: now also N2.2 (C), N3.1 (A); no longer J3.3 (Pin_3), J4.19
- new net SERVO_GND: J3.3 (Pin_3), J4.19, N3.2 (C)
Other:
- sheet MCU ports: added DATA_0, DATA_1, DATA_2, DATA_3, DATA_4, DATA_5, DATA_6, DATA_7, LIMIT_SWITCH_IN, SCK_OUT, SERVO_PWM_OUT; removed DT1, DT2, DT3, DT4, DT5, DT6, DT7, DT8, LIMIT_SWITCH, SCK, SERVO_PWM_OUTPUT
- moved on the sheet: N2
