File: truss_connector_breakout/truss_connector_breakout.kicad_sch (KiCad schematic)
At the start: 10 parts, among them J1 D3, J10 Truss Connector, J2 D4, J3 Servo, J4 D5, J5 D6/LC, J6 LimitSwitch, J7 D0, J8 D1, J9 D2

Commit message: update
Parts:
- removed J1: D3, TerminalBlock_WAGO:TerminalBlock_WAGO_236-204_1x04_P7.50mm_45Degree, symbol 000_Connectors_Immo:Wago_01x04_cage_clamp
- removed J2: D4, TerminalBlock_WAGO:TerminalBlock_WAGO_236-204_1x04_P7.50mm_45Degree, symbol 000_Connectors_Immo:Wago_01x04_cage_clamp
- removed J4: D5, TerminalBlock_WAGO:TerminalBlock_WAGO_236-204_1x04_P7.50mm_45Degree, symbol 000_Connectors_Immo:Wago_01x04_cage_clamp
- removed J5: D6/LC, TerminalBlock_WAGO:TerminalBlock_WAGO_236-204_1x04_P7.50mm_45Degree, symbol 000_Connectors_Immo:Wago_01x04_cage_clamp
- removed J7: D0, TerminalBlock_WAGO:TerminalBlock_WAGO_236-204_1x04_P7.50mm_45Degree, symbol 000_Connectors_Immo:Wago_01x04_cage_clamp
- removed J8: D1, TerminalBlock_WAGO:TerminalBlock_WAGO_236-204_1x04_P7.50mm_45Degree, symbol 000_Connectors_Immo:Wago_01x04_cage_clamp
- removed J9: D2, TerminalBlock_WAGO:TerminalBlock_WAGO_236-204_1x04_P7.50mm_45Degree, symbol 000_Connectors_Immo:Wago_01x04_cage_clamp
- added H1, H2, H3, H4: MountingHole_M3, MountingHole:MountingHole_3.2mm_M3_Pad_Via, symbol Mechanical:MountingHole_M3
- added J1: D3, TerminalBlock_Phoenix:TerminalBlock_Phoenix_MPT-0,5-4-2.54_1x04_P2.54mm_Horizontal, symbol 000_Connectors_Immo:pheonix_01x04_screwterminal_2.54mm
- added J2: D4, TerminalBlock_Phoenix:TerminalBlock_Phoenix_MPT-0,5-4-2.54_1x04_P2.54mm_Horizontal, symbol 000_Connectors_Immo:pheonix_01x04_screwterminal_2.54mm
- added J4: D5, TerminalBlock_Phoenix:TerminalBlock_Phoenix_MPT-0,5-4-2.54_1x04_P2.54mm_Horizontal, symbol 000_Connectors_Immo:pheonix_01x04_screwterminal_2.54mm
- added J5: D6, TerminalBlock_Phoenix:TerminalBlock_Phoenix_MPT-0,5-4-2.54_1x04_P2.54mm_Horizontal, symbol 000_Connectors_Immo:pheonix_01x04_screwterminal_2.54mm
- added J7: D0, TerminalBlock_Phoenix:TerminalBlock_Phoenix_MPT-0,5-4-2.54_1x04_P2.54mm_Horizontal, symbol 000_Connectors_Immo:pheonix_01x04_screwterminal_2.54mm
- added J8: D1, TerminalBlock_Phoenix:TerminalBlock_Phoenix_MPT-0,5-4-2.54_1x04_P2.54mm_Horizontal, symbol 000_Connectors_Immo:pheonix_01x04_screwterminal_2.54mm
- added J9: D2, TerminalBlock_Phoenix:TerminalBlock_Phoenix_MPT-0,5-4-2.54_1x04_P2.54mm_Horizontal, symbol 000_Connectors_Immo:pheonix_01x04_screwterminal_2.54mm
- J10: footprint Connector_Dsub:DSUB-37_Female_Vertical_P2.77x2.84mm_MountingHoles -> Connector_Dsub:DSUB-37_Male_Horizontal_P2.77x2.84mm_EdgePinOffset9.90mm_Housed_MountingHolesOffset11.32mm
- J6: footprint TerminalBlock_WAGO:TerminalBlock_WAGO_236-102_1x02_P5.00mm_45Degree -> TerminalBlock_Phoenix:TerminalBlock_Phoenix_MPT-0,5-2-2.54_1x02_P2.54mm_Horizontal
Connections:
- net D0_GND: now also J7.3 (Pin_3)
- net D0_LC+: now also J7.1 (Pin_1)
- net D0_LC-: now also J7.2 (Pin_2)
- net D0_VCC: now also J7.4 (Pin_4)
- net D1_GND: now also J8.3 (Pin_3)
- net D1_LC+: now also J8.1 (Pin_1)
- net D1_LC-: now also J8.2 (Pin_2)
- net D1_VCC: now also J8.4 (Pin_4)
- net D2_GND: now also J9.3 (Pin_3)
- net D2_LC+: now also J9.1 (Pin_1)
- net D2_LC-: now also J9.2 (Pin_2)
- net D2_VCC: now also J9.4 (Pin_4)
- net D3_GND: now also J1.3 (Pin_3)
- net D3_LC+: now also J1.1 (Pin_1)
- net D3_LC-: now also J1.2 (Pin_2)
- net D3_VCC: now also J1.4 (Pin_4)
- net D4_GND: now also J2.3 (Pin_3)
- net D4_LC+: now also J2.1 (Pin_1)
- net D4_LC-: now also J2.2 (Pin_2)
- net D4_VCC: now also J2.4 (Pin_4)
- net D5_GND: now also J4.3 (Pin_3)
- net D5_LC+: now also J4.1 (Pin_1)
- net D5_LC-: now also J4.2 (Pin_2)
- net D5_VCC: now also J4.4 (Pin_4)
- net D6_GND: now also J5.3 (Pin_3)
- net D6_LC+: now also J5.1 (Pin_1)
- net D6_LC-: now also J5.2 (Pin_2)
- net D6_VCC: now also J5.4 (Pin_4)
- net LIMIT_SWITCH: now also J6.2 (Pin_2); no longer J6.1 (Pin_1)
- net LS_GND: now also J6.1 (Pin_1); no longer J6.2 (Pin_2)
