File: truss_PCB/bridge_driver0_sch.kicad_sch (KiCad schematic)
At the start: 16 parts, among them J5 IN_B, Q1 BC807, U1 HX711

Commit message: updating truss PCB
Parts:
- renumbered C1 to C16, C2 to C17, C3 to C18, EC1 to EC11, EC2 to EC12, J5 to J10, JP2 to JP17, JP3 to JP18, JP4 to JP19, Q1 to Q6, R2 to R27, R3 to R28, R4 to R29, R5 to R30, R6 to R31, U1 to U6
Changed lines of the file:
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@@
   (symbol (lib_id "000_Capacitor_Film_Immo:cap_film_0805") (at 209.55 80.01 0)
     (in_bom yes) (on_board yes) (fields_autoplaced)
-    (property "Reference" "C3" (id 0) (at 212.725 78.7399 0)
+    (property "Reference" "C18" (id 0) (at 212.725 78.7399 0)
       (effects (font (size 1.27 1.27)) (justify left))
     )
@@
   (symbol (lib_id "Transistor_BJT:BC807") (at 108.585 72.39 180)
     (in_bom yes) (on_board yes)
-    (property "Reference" "Q1" (id 0) (at 104.14 67.945 0)
+    (property "Reference" "Q6" (id 0) (at 104.14 67.945 0)
       (effects (font (size 1.27 1.27)) (justify left))
     )
@@
   (symbol (lib_id "000_Capacitor_Film_Immo:cap_film_0805") (at 144.145 99.695 90)
     (in_bom yes) (on_board yes)
-    (property "Reference" "C2" (id 0) (at 142.24 104.14 0)
+    (property "Reference" "C17" (id 0) (at 142.24 104.14 0)
       (effects (font (size 1.27 1.27)) (justify left))
     )
@@
   (symbol (lib_id "000_Pin_Headers_Immo:Conn_01x02_Male") (at 191.77 91.44 180)
     (in_bom yes) (on_board yes) (fields_autoplaced)
-    (property "Reference" "J5" (id 0) (at 193.675 88.8999 0)
+    (property "Reference" "J10" (id 0) (at 193.675 88.8999 0)
       (effects (font (size 1.27 1.27)) (justify right))
     )
@@
   (symbol (lib_id "000_Resistors_Immo:Resistor_0805") (at 133.35 113.03 180)
     (in_bom yes) (on_board yes)
-    (property "Reference" "R5" (id 0) (at 132.715 115.57 0))
+    (property "Reference" "R30" (id 0) (at 132.715 115.57 0))
     (property "Value" "100r" (id 1) (at 133.35 117.475 0))
     (property "Footprint" "Resistor_SMD:R_0805_2012Metric_Pad1.20x1.40mm_HandSolder" (id 2) (at 133.35 111.252 0)
@@
   (symbol (lib_id "000_Sensors_Immo:HX711_24bit_ADC_Strain_Gauge_Driver") (at 158.115 78.74 0)
     (in_bom yes) (on_board yes)
-    (property "Reference" "U1" (id 0) (at 161.925 56.515 0))
+    (property "Reference" "U6" (id 0) (at 161.925 56.515 0))
     (property "Value" "HX711" (id 1) (at 161.925 59.055 0))
     (property "Footprint" "Package_SO:SOP-16_4.55x10.3mm_P1.27mm" (id 2) (at 148.59 109.855 0)
@@
   (symbol (lib_id "000_Resistors_Immo:Resistor_0805") (at 106.045 95.25 90)
     (in_bom yes) (on_board yes) (fields_autoplaced)
-    (property "Reference" "R3" (id 0) (at 107.95 93.9799 90)
+    (property "Reference" "R28" (id 0) (at 107.95 93.9799 90)
       (effects (font (size 1.27 1.27)) (justify right))
     )
@@
   (symbol (lib_id "000_Connectors_Immo:Jumper_3_BridgeSmall") (at 177.165 96.52 180)
     (in_bom yes) (on_board yes) (fields_autoplaced)
-    (property "Reference" "JP3" (id 0) (at 173.99 95.7579 0)
+    (property "Reference" "JP18" (id 0) (at 173.99 95.7579 0)
       (effects (font (size 1.27 1.27)) (justify left))
     )
@@
   (symbol (lib_id "000_Resistors_Immo:Resistor_0805") (at 106.045 85.725 90)
     (in_bom yes) (on_board yes) (fields_autoplaced)
-    (property "Reference" "R2" (id 0) (at 107.95 84.4549 90)
+    (property "Reference" "R27" (id 0) (at 107.95 84.4549 90)
       (effects (font (size 1.27 1.27)) (justify right))
     )
@@
   (symbol (lib_id "000_Resistors_Immo:Resistor_0805") (at 133.35 109.855 180)
     (in_bom yes) (on_board yes)
-    (property "Reference" "R4" (id 0) (at 132.715 105.41 0))
+    (property "Reference" "R29" (id 0) (at 132.715 105.41 0))
     (property "Value" "100r" (id 1) (at 133.35 107.315 0))
     (property "Footprint" "Resistor_SMD:R_0805_2012Metric_Pad1.20x1.40mm_HandSolder" (id 2) (at 133.35 108.077 0)
@@
   (symbol (lib_id "000_Capacitor_Film_Immo:cap_film_0805") (at 135.255 95.885 0)
     (in_bom yes) (on_board yes)
-    (property "Reference" "C1" (id 0) (at 130.81 93.98 0)
+    (property "Reference" "C16" (id 0) (at 130.81 93.98 0)
       (effects (font (size 1.27 1.27)) (justify left))
     )
@@
   (symbol (lib_id "000_Connectors_Immo:Jumper_2_Bridge_Small") (at 122.555 75.565 180)
     (in_bom yes) (on_board yes)
-    (property "Reference" "JP2" (id 0) (at 123.19 73.66 0))
+    (property "Reference" "JP17" (id 0) (at 123.19 73.66 0))
     (property "Value" "Gain" (id 1) (at 123.19 78.105 0))
     (property "Footprint" "Jumper:SolderJumper-2_P1.3mm_Bridged_RoundedPad1.0x1.5mm" (id 2) (at 121.92 69.85 0)
@@
   (symbol (lib_id "000_Capacitor_Electrolytic_Immo:22u") (at 221.615 80.01 0)
     (in_bom yes) (on_board yes) (fields_autoplaced)
-    (property "Reference" "EC2" (id 0) (at 225.425 77.8509 0)
+    (property "Reference" "EC12" (id 0) (at 225.425 77.8509 0)
       (effects (font (size 1.27 1.27)) (justify left))
     )
@@
   (symbol (lib_id "000_Connectors_Immo:Jumper_2_Bridge_Small") (at 187.96 74.93 90)
     (in_bom yes) (on_board yes) (fields_autoplaced)
-    (property "Reference" "JP4" (id 0) (at 189.865 73.9998 90)
+    (property "Reference" "JP19" (id 0) (at 189.865 73.9998 90)
       (effects (font (size 1.27 1.27)) (justify right))
     )
@@
   (symbol (lib_id "000_Resistors_Immo:Resistor_0805") (at 187.96 67.31 270)
     (in_bom yes) (on_board yes)
-    (property "Reference" "R6" (id 0) (at 183.515 67.945 0))
+    (property "Reference" "R31" (id 0) (at 183.515 67.945 0))
     (property "Value" "10k" (id 1) (at 185.42 67.31 0))
     (property "Footprint" "Resistor_SMD:R_0805_2012Metric_Pad1.20x1.40mm_HandSolder" (id 2) (at 186.182 67.31 0)
@@
   (symbol (lib_id "000_Capacitor_Electrolytic_Immo:22u") (at 93.98 90.17 0)
     (in_bom yes) (on_board yes) (fields_autoplaced)
-    (property "Reference" "EC1" (id 0) (at 97.79 88.0109 0)
-      (effects (font (size 1.27 1.27)) (justify left))
-    )
+    (property "Reference" "EC11" (id 0) (at 97.79 88.0109 0)
+      (effects (font (size 1.27 1.27)) (justify left))
+    )

Commit message: Finished PCB Version 2 Design
Parts:
- renumbered C16 to C7, C17 to C8, C18 to C9, EC11 to EC5, EC12 to EC6, J10 to J7, JP19 to JP10, JP17 to JP8, JP18 to JP9, Q6 to Q3, R27 to R12, R28 to R13, R29 to R14, R30 to R15, R31 to R16, U6 to U3
Changed lines of the file:
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@@
   (symbol (lib_id "000_Capacitor_Film_Immo:cap_film_0805") (at 209.55 80.01 0)
     (in_bom yes) (on_board yes) (fields_autoplaced)
-    (property "Reference" "C18" (id 0) (at 212.725 78.7399 0)
+    (property "Reference" "C9" (id 0) (at 212.725 78.7399 0)
       (effects (font (size 1.27 1.27)) (justify left))
     )
@@
   (symbol (lib_id "Transistor_BJT:BC807") (at 108.585 72.39 180)
     (in_bom yes) (on_board yes)
-    (property "Reference" "Q6" (id 0) (at 104.14 67.945 0)
+    (property "Reference" "Q3" (id 0) (at 104.14 67.945 0)
       (effects (font (size 1.27 1.27)) (justify left))
     )
@@
   (symbol (lib_id "000_Capacitor_Film_Immo:cap_film_0805") (at 144.145 99.695 90)
     (in_bom yes) (on_board yes)
-    (property "Reference" "C17" (id 0) (at 142.24 104.14 0)
+    (property "Reference" "C8" (id 0) (at 142.24 104.14 0)
       (effects (font (size 1.27 1.27)) (justify left))
     )
@@
   (symbol (lib_id "000_Pin_Headers_Immo:Conn_01x02_Male") (at 191.77 91.44 180)
     (in_bom yes) (on_board yes) (fields_autoplaced)
-    (property "Reference" "J10" (id 0) (at 193.675 88.8999 0)
+    (property "Reference" "J7" (id 0) (at 193.675 88.8999 0)
       (effects (font (size 1.27 1.27)) (justify right))
     )
@@
   (symbol (lib_id "000_Resistors_Immo:Resistor_0805") (at 133.35 113.03 180)
     (in_bom yes) (on_board yes)
-    (property "Reference" "R30" (id 0) (at 132.715 115.57 0))
+    (property "Reference" "R15" (id 0) (at 132.715 115.57 0))
     (property "Value" "100r" (id 1) (at 133.35 117.475 0))
     (property "Footprint" "Resistor_SMD:R_0805_2012Metric_Pad1.20x1.40mm_HandSolder" (id 2) (at 133.35 111.252 0)
@@
   (symbol (lib_id "000_Sensors_Immo:HX711_24bit_ADC_Strain_Gauge_Driver") (at 158.115 78.74 0)
     (in_bom yes) (on_board yes)
-    (property "Reference" "U6" (id 0) (at 161.925 56.515 0))
+    (property "Reference" "U3" (id 0) (at 161.925 56.515 0))
     (property "Value" "HX711" (id 1) (at 161.925 59.055 0))
     (property "Footprint" "Package_SO:SOP-16_4.55x10.3mm_P1.27mm" (id 2) (at 148.59 109.855 0)
@@
   (symbol (lib_id "000_Resistors_Immo:Resistor_0805") (at 106.045 95.25 90)
     (in_bom yes) (on_board yes) (fields_autoplaced)
-    (property "Reference" "R28" (id 0) (at 107.95 93.9799 90)
+    (property "Reference" "R13" (id 0) (at 107.95 93.9799 90)
       (effects (font (size 1.27 1.27)) (justify right))
     )
@@
   (symbol (lib_id "000_Connectors_Immo:Jumper_3_BridgeSmall") (at 177.165 96.52 180)
     (in_bom yes) (on_board yes) (fields_autoplaced)
-    (property "Reference" "JP18" (id 0) (at 173.99 95.7579 0)
+    (property "Reference" "JP9" (id 0) (at 173.99 95.7579 0)
       (effects (font (size 1.27 1.27)) (justify left))
     )
@@
   (symbol (lib_id "000_Resistors_Immo:Resistor_0805") (at 106.045 85.725 90)
     (in_bom yes) (on_board yes) (fields_autoplaced)
-    (property "Reference" "R27" (id 0) (at 107.95 84.4549 90)
+    (property "Reference" "R12" (id 0) (at 107.95 84.4549 90)
       (effects (font (size 1.27 1.27)) (justify right))
     )
@@
   (symbol (lib_id "000_Resistors_Immo:Resistor_0805") (at 133.35 109.855 180)
     (in_bom yes) (on_board yes)
-    (property "Reference" "R29" (id 0) (at 132.715 105.41 0))
+    (property "Reference" "R14" (id 0) (at 132.715 105.41 0))
     (property "Value" "100r" (id 1) (at 133.35 107.315 0))
     (property "Footprint" "Resistor_SMD:R_0805_2012Metric_Pad1.20x1.40mm_HandSolder" (id 2) (at 133.35 108.077 0)
@@
   (symbol (lib_id "000_Capacitor_Film_Immo:cap_film_0805") (at 135.255 95.885 0)
     (in_bom yes) (on_board yes)
-    (property "Reference" "C16" (id 0) (at 130.81 93.98 0)
+    (property "Reference" "C7" (id 0) (at 130.81 93.98 0)
       (effects (font (size 1.27 1.27)) (justify left))
     )
@@
   (symbol (lib_id "000_Connectors_Immo:Jumper_2_Bridge_Small") (at 122.555 75.565 180)
     (in_bom yes) (on_board yes)
-    (property "Reference" "JP17" (id 0) (at 123.19 73.66 0))
+    (property "Reference" "JP8" (id 0) (at 123.19 73.66 0))
     (property "Value" "Gain" (id 1) (at 123.19 78.105 0))
     (property "Footprint" "Jumper:SolderJumper-2_P1.3mm_Bridged_RoundedPad1.0x1.5mm" (id 2) (at 121.92 69.85 0)
@@
   (symbol (lib_id "000_Capacitor_Electrolytic_Immo:22u") (at 221.615 80.01 0)
     (in_bom yes) (on_board yes) (fields_autoplaced)
-    (property "Reference" "EC12" (id 0) (at 225.425 77.8509 0)
+    (property "Reference" "EC6" (id 0) (at 225.425 77.8509 0)
       (effects (font (size 1.27 1.27)) (justify left))
     )
@@
   (symbol (lib_id "000_Connectors_Immo:Jumper_2_Bridge_Small") (at 187.96 74.93 90)
     (in_bom yes) (on_board yes) (fields_autoplaced)
-    (property "Reference" "JP19" (id 0) (at 189.865 73.9998 90)
+    (property "Reference" "JP10" (id 0) (at 189.865 73.9998 90)
       (effects (font (size 1.27 1.27)) (justify right))
     )
@@
   (symbol (lib_id "000_Resistors_Immo:Resistor_0805") (at 187.96 67.31 270)
     (in_bom yes) (on_board yes)
-    (property "Reference" "R31" (id 0) (at 183.515 67.945 0))
+    (property "Reference" "R16" (id 0) (at 183.515 67.945 0))
     (property "Value" "10k" (id 1) (at 185.42 67.31 0))
     (property "Footprint" "Resistor_SMD:R_0805_2012Metric_Pad1.20x1.40mm_HandSolder" (id 2) (at 186.182 67.31 0)
@@
   (symbol (lib_id "000_Capacitor_Electrolytic_Immo:22u") (at 93.98 90.17 0)
     (in_bom yes) (on_board yes) (fields_autoplaced)
-    (property "Reference" "EC11" (id 0) (at 97.79 88.0109 0)
-      (effects (font (size 1.27 1.27)) (justify left))
-    )
+    (property "Reference" "EC5" (id 0) (at 97.79 88.0109 0)
+      (effects (font (size 1.27 1.27)) (justify left))
+    )
