File: truss_PCB/micro_controller_sch.kicad_sch (KiCad schematic)
At the start: 39 parts, among them J12 Serial IO, J13 IO Header, J14 LV IO, J15 HV IO, U8 TXS0108EPW, U9 TXS0108EPW

Commit message: updating truss PCB
Parts:
- added R47, R48, R49, R50, R51: 10k, Resistor_SMD:R_0805_2012Metric_Pad1.20x1.40mm_HandSolder, symbol 000_Resistors_Immo:Resistor_0805
Connections:
- net DGND: now also R47.1, R48.1, R49.1, R50.1, R51.1
- net at J14.1 (Pin_1), U8.5 (A4): now also R47.2
- net at J14.2 (Pin_2), U8.6 (A5): now also R48.2
- net at J14.3 (Pin_3), U8.7 (A6): now also R49.2
- net at J14.4 (Pin_4), U8.8 (A7): now also R50.2
- net at J14.5 (Pin_5), U8.9 (A8): now also R51.2
- net LED_2: now reaches A1.24 (A5), D9.2 (A), J13.5 (Pin_5)
- net TX: now reaches A1.1 (D1/TX), J12.5 (Pin_5)
- net RX: now reaches A1.2 (D0/RX), J12.4 (Pin_4)
- net LED_3: now reaches A1.25 (A6), D10.2 (A), J13.6 (Pin_6)
- net LED_4: now reaches A1.26 (A7), D11.2 (A), J13.7 (Pin_7)
- net SPARE_0 renamed LED_1
Other:
- moved on the sheet: D1, D10, D11, D9, J14, R37, R44, R45, R46

Commit message: Finished PCB Version 2 Design
Other:
- moved on the sheet: R47, R48, R49, R50, R51
